File: PCB/WaifuFC.kicad_pcb (KiCad board)
At the start: 4 copper layers, 40.2 x 38.1 mm, 58 parts, among them J1 SBUS, J2 USB_C_Receptacle_USB2.0, J3 PPM, J4 OUT, J5 Conn_01x02, J6 Conn_01x02, J7 Conn_01x04, Q1 1P, SW1 SW_Push, U1 STM32F103C8Tx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

Commit message: fixes
Parts:
- moved D3 6.11 mm to (127.3, 85.4)
- moved D4 6.11 mm to (129.0, 85.4)
- moved D5 6.11 mm to (130.7, 85.4)
- moved R17 5.26 mm to (126.5, 90.2)
- moved C5 5.26 mm to (127.8, 90.2)
- moved R15 5.26 mm to (124.0, 90.2)
- moved R16 5.26 mm to (125.2, 90.2)
- moved C10 4.00 mm to (135.0, 90.3), turned to 90 degrees
- moved C17 3.36 mm to (158.5, 106.9)
- moved C1 3.20 mm to (130.7, 93.8)
- moved C6 3.20 mm to (126.4, 92.7)
- moved C7 3.20 mm to (130.6, 92.7)
- moved R1 3.20 mm to (126.4, 93.8)
- moved R18 3.20 mm to (128.6, 93.8)
- moved R19 3.20 mm to (128.6, 92.7)
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Routing:
- net +5V: track 56.4 -> 142.1 mm, vias 1 -> 3
- net /USB_DN: track 0.00 -> 40.6 mm, vias 0 -> 4
- net GND: track 213.9 -> 239.7 mm, vias 4 -> 5
- net /VBAT: track 8.79 -> 33.4 mm
- net /BST: track 9.04 -> 32.6 mm
- net /LED_STATUS: track 17.5 -> 40.5 mm
- net /REGOUT: track 17.0 -> 38.8 mm, vias 0 -> 2
- net /IMU_SCL: track 1.56 -> 16.6 mm, vias 1 -> 3
- net Net-(D4-Pad2): track 1.83 -> 14.1 mm
- net /TIM3_S3: track 16.3 -> 27.9 mm
- net /HSE_IN: track 33.9 -> 44.8 mm, vias 3 -> 4
- net /TIM3_S2: track 20.5 -> 31.2 mm, vias 1 -> 2
- net +3V3: track 135.1 -> 124.5 mm, vias 6 -> 4
- net /HSE_OUT: track 7.50 -> 18.0 mm, vias 0 -> 3
- net /IMU_SDA: track 15.9 -> 26.1 mm
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Other:
- copper layers 4 -> 2

Commit message: v3
Parts:
- added G***: LOGO, SFA_LOGO:Arrow, F.Cu at (145.7, 89.3)
- added R20: R, Resistor_SMD:R_0402_1005Metric, F.Cu at (143.9, 81.8)
- added R21: R, Resistor_SMD:R_0402_1005Metric, F.Cu at (145.9, 81.8)
- moved J5 39.1 mm to (121.0, 89.1), turned to 0 degrees
- moved J6 21.1 mm to (124.8, 115.7), turned to -90 degrees
- moved C11 15.6 mm to (136.4, 86.4)
- moved C9 12.9 mm to (136.8, 78.7)
- moved C8 12.9 mm to (138.1, 78.7)
- moved R3 12.0 mm to (140.2, 86.5)
- moved U2 12.0 mm to (137.2, 82.6)
- moved R4 11.8 mm to (139.1, 86.4)
- moved C2 11.3 mm to (134.7, 89.2)
- moved J7 11.2 mm to (143.3, 78.8)
- moved R17 9.83 mm to (131.6, 81.8)
- moved R16 9.61 mm to (129.9, 81.8)
- moved R15 9.39 mm to (128.2, 81.8)
- moved J3 9.38 mm to (158.4, 107.9)
- moved R18 9.33 mm to (125.8, 102.7)
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Connections:
- J2 pad A5: unconnected-(J2-PadA5) -> Net-(J2-CC1)
- J2 pad B5: unconnected-(J2-PadB5) -> Net-(J2-CC2)
Routing:
- net +3V3: track 124.5 -> 176.8 mm, vias 4 -> 5
- net /REGOUT: track 38.8 -> 1.53 mm, vias 2 -> 0
- net /HSE_IN: track 44.8 -> 10.5 mm, vias 4 -> 0
- net /USB_DN: track 40.6 -> 6.87 mm, vias 4 -> 0
- net GND: track 239.7 -> 265.5 mm, vias 5 -> 1
- net +5V: track 142.1 -> 116.6 mm, vias 3 -> 2
- net /LED_STATUS: track 40.5 -> 17.3 mm
- net Net-(J2-CC1): track 0.00 -> 21.6 mm, vias 0 -> 2
- net /IMU_SDA: track 26.1 -> 9.76 mm
- net GNDPWR: track 57.7 -> 74.0 mm, vias 0 -> 1
- net Net-(J2-CC2): track 0.00 -> 16.1 mm
- net /USB_DP: track 20.3 -> 6.87 mm, vias 2 -> 0
- net Net-(D4-A): track 14.1 -> 1.43 mm
- net /VIN: track 26.0 -> 38.2 mm
- net /TIM3_S2: track 31.2 -> 19.0 mm, vias 2 -> 1
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Other:
- board size 40.2 x 38.1 mm -> 40 x 40 mm

Commit message: elowina
Parts:
- R20, R21: value R -> 5.1k
- moved NT1 32.3 mm to (154.4, 112.9)
- moved Q1 6.00 mm to (146.4, 88.0)
- moved C12 5.48 mm to (119.7, 109.2)
- moved R13 5.35 mm to (129.7, 100.3)
- moved R2 4.92 mm to (118.8, 104.9)
- moved R12 3.98 mm to (134.4, 102.3)
- moved R11 3.82 mm to (122.7, 104.2)
- moved D2 3.78 mm to (138.0, 105.5)
- moved U3 3.54 mm to (128.2, 106.9)
- moved C13 3.44 mm to (134.4, 104.0)
- moved C16 3.36 mm to (148.2, 102.1)
- moved R17 3.11 mm to (131.9, 84.9)
- moved R9 2.75 mm to (134.4, 106.2)
- moved R10 2.57 mm to (134.3, 107.9)
- moved R16 2.50 mm to (129.8, 84.3)
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Routing:
- net +3V3: track 176.8 -> 220.1 mm, vias 5 -> 1
- net +5V: track 116.6 -> 147.8 mm, vias 2 -> 1
- net /BOOT: track 23.8 -> 52.0 mm
- net /NRST: track 15.2 -> 39.0 mm, vias 0 -> 2
- net /BST: track 32.9 -> 12.6 mm
- net /TIM3_S3: track 19.5 -> 38.4 mm, vias 1 -> 3
- net GNDPWR: track 74.0 -> 91.7 mm
- net GND: track 265.5 -> 249.4 mm, vias 1 -> 2
- net Net-(J2-CC2): track 16.1 -> 29.8 mm
- net /VIN: track 38.2 -> 25.9 mm
- net /TIM3_S2: track 19.0 -> 29.8 mm
- net /IMU_INT: track 13.6 -> 23.7 mm
- net /VBAT: track 30.0 -> 39.5 mm, vias 2 -> 0
- net /SW: track 11.9 -> 20.5 mm
- net /SWDIO: track 28.4 -> 20.4 mm, vias 3 -> 1
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Other:
- board size 40 x 40 mm -> 43.6 x 43.2 mm
